File: GSR_v1.sch (KiCad schematic (older format))
At the start: 63 parts, among them P1 CONN_2, P2 CONN_2, P3 CONN_2, P4 CONN_2, Q1 DMP21D5UFB4-7B, U1 TPS63001, U2 LM324N, U3 NRF528XX-QFAA, U4 TMP116, U5 TPS2294x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

Commit message: Upgraded to KiCAD 5.0 compat
Parts:
- A1: symbol CHIP-ANT -> conn1:CHIP-ANT
- C1, C14, C15, C16, C17, C18, C2, C21, C22, C23, C24, C25, C26, C27, C28, C29, C3, C30, C33, C34, C4, C5, C6: symbol C -> Device:C
- D3: symbol LED-RESCUE-EEG_ADS1299_2 -> EEG_ADS1299_2-cache:LED-RESCUE-EEG_ADS1299_2
- D4: symbol D_Schottky -> Device:D_Schottky
- F1: symbol 2450FM07A0029 -> EEG_ADS1299_2-cache:2450FM07A0029
- L1, L3, L4, L5, L6: symbol INDUCTOR -> conn1:INDUCTOR
- P1, P2, P3, P4: symbol CONN_2 -> conn1:CONN_2
- Q1: symbol Q_PMOS_GDS -> Device:Q_PMOS_GDS
- R1, R10, R11, R12, R13, R14, R15, R16, R17, R18, R2, R3, R4, R5, R6, R7, R8, R9: symbol R -> Device:R
- U1: symbol TPS63001 -> EEG_ADS1299_2-cache:TPS63001
- U2: symbol LM324N -> GSR_v1-rescue:LM324N
- U3: symbol NRF528XX-QFAA-RESCUE-EEG_ADS1299_2 -> EEG_ADS1299_2-cache:NRF528XX-QFAA-RESCUE-EEG_ADS1299_2
- U4: symbol TMP116 -> GSR_v1-rescue:TMP116
- U5: symbol TPS2294x -> EEG_ADS1299_2-cache:TPS2294x
- U6: symbol MCP73831 -> EEG_ADS1299_2-cache:MCP73831
- X1: symbol Crystal_GND24 -> Device:Crystal_GND24
- X2: symbol Crystal -> Device:Crystal
Connections:
- wire segments 261 -> 319

Commit message: Major refactoring and cleanup.
Connections:
- wire segments 319 -> 317
Other:
- note added: "3.3V Voltage Regulator, 2A Max output"
- note added: "GSR Analog Front End"
- note added: "LOAD_IN = Vcc = Battery Voltage"
- note added: "Load Switch for Battery Measurement with Voltage Divider (V/2)"
- note added: "Pin Headers and General Connection Labeling"
- note added: "Power Regulation Circuitry"
- note added: "Q1 = DMP21D5UFB4 P-mosfet\nFootprint: X2-DFN1006-3"
- note added: "Recharge Circuitry"
- note added: "Temperature Sensor IC"
- note added: "nRF52 Module"
- note removed: "Configuration for EEG and EMG different\nFor EEG, only channels 1-4 used\nUnused to AVDD"
- note removed: "Power Regulation Circuit"
- note removed: "Q1 = DMP21D5UFB4 P-mosfet\nCase: X2-DFN1006-3"
- note removed: "Remember to Annotate"
- note removed: "Remove switch??"

Commit message: Updated Gerbers, deleted old gerber files, minor details. Updated silkscreen (back)
Other:
- note added: "GSR Analog Front End (Using 4-Op Amp LM324-N Configured as Instrumentation Amp)"
- note removed: "GSR Analog Front End"
Changed lines of the file:
@@
 	20900 12200 20900 8250
 Text Notes 20900 8250 0    50   ~ 0
-GSR Analog Front End
+GSR Analog Front End (Using 4-Op Amp LM324-N Configured as Instrumentation Amp)
 Wire Notes Line
 	20600 8250 20600 12200

Commit message: moved connectors for Temp sensor down to make space for uSD card
Parts:
- added J1: Micro_SD_Card, symbol Connector:Micro_SD_Card
Connections:
- net labels added: CMD, DAT0, DAT1, DAT2, DAT3, uSD_CLK
- wire segments 317 -> 330
Changed lines of the file:
@@
 Text GLabel 22000 4450 3    60   Input ~ 0
 DGND
-Text Label 24500 6150 0    60   ~ 0
-SCL
-Text Label 24700 6000 0    60   ~ 0
-SDA
 $Comp
 L EEG_ADS1299_2-cache:TPS63001 U1
@@
 	22400 4450 22000 4450
 Wire Wire Line
-	24300 5700 24300 6150
-Wire Wire Line
-	24300 6150 24500 6150
-Wire Wire Line
-	24400 5700 24400 6000
-Wire Wire Line
-	24400 6000 24700 6000
-Wire Wire Line
 	17050 1700 17050 2350
 Wire Wire Line
@@
 	18300 11150 18100 11150
 Connection ~ 18100 11150
-Text Label 24250 6300 0    60   ~ 0
-ALERT
-Wire Wire Line
-	24200 5700 24200 6300
-Wire Wire Line
-	24200 6300 24250 6300
 Wire Wire Line
 	29100 4000 29150 4000
@@
 Text Notes 2750 1150 0    50   ~ 0
 Pin Headers and General Connection Labeling
+$Comp
+L Connector:Micro_SD_Card J1
+U 1 1 5C383B9E
+P 10700 10350
+F 0 "J1" H 10650 9533 50  0000 C CNN
+F 1 "Micro_SD_Card" H 10650 9624 50  0000 C CNN
+F 2 "" H 11850 10650 50  0001 C CNN
+F 3 "http://katalog.we-online.de/em/datasheet/693072010801.pdf" H 10700 10350 50  0001 C CNN
+	1    10700 10350
+	-1   0    0    1
+$EndComp
+Wire Notes Line
+	15400 8250 9150 8250
+Wire Notes Line
+	9150 8250 9150 12200
+Wire Notes Line
+	9150 12200 15400 12200
+Wire Notes Line
+	15400 12200 15400 8250
+Wire Wire Line
+	11600 10150 11950 10150
+Wire Wire Line
+	11950 10150 11950 9300
+Wire Wire Line
+	11950 9300 9800 9300
+Wire Wire Line
+	9800 9300 9800 9750
+Wire Wire Line
+	9800 9750 9900 9750
+Wire Wire Line
+	11600 9950 12400 9950
+Wire Wire Line
+	11600 10050 12400 10050
+Text Label 12400 9950 0    50   ~ 0
+DAT1
+Text Label 12400 10050 0    50   ~ 0
+DAT0
+Wire Wire Line
+	11950 9300 12250 9300
+Connection ~ 11950 9300
+Text GLabel 12250 9300 2    60   Input ~ 0
+DGND
+Wire Wire Line
+	11600 10250 12700 10250
+Text Label 12700 10250 0    50   ~ 0
+uSD_CLK
+Wire Wire Line
+	13100 10350 13100 9300
+Wire Wire Line
+	11600 10350 13100 10350
+Text GLabel 13100 9300 2    60   Input ~ 0
+DVDD
+Wire Wire Line
+	11600 10450 12400 10450
+Text Label 12400 10450 0    50   ~ 0
+CMD
+Wire Wire Line
+	11600 10550 12400 10550
+Text Label 12400 10550 0    50   ~ 0
+DAT3
+Wire Wire Line
+	11600 10650 12400 10650
+Text Label 12400 10650 0    50   ~ 0
+DAT2
+Wire Wire Line
+	25050 4800 25550 4800
+Wire Wire Line
+	25550 4800 25550 5400
+Wire Wire Line
+	23400 5700 23400 6250
+Wire Wire Line
+	23500 5700 23500 6250
+Wire Wire Line
+	23600 5700 23600 6250
+Text Label 23400 6250 1    60   ~ 0
+ALERT
+Text Label 23500 6250 1    60   ~ 0
+SCL
+Text Label 23600 6250 1    60   ~ 0
+SDA
 $EndSCHEMATC

Commit message: Added microSD Card to sch and pcb
Parts:
- removed J1: Micro_SD_Card, symbol Connector:Micro_SD_Card
- added J1: Micro_SD_Card_Det, symbol Connector:Micro_SD_Card_Det
Connections:
- net labels added: CMD_MOSI, DAT0_MISO, DAT1_UNUSED, DAT2_UNUSED, DAT3_CS
- net labels removed: CMD, DAT0, DAT1, DAT2, DAT3
- wire segments 330 -> 337
- no-connect marks 1 -> 3
Other:
- note added: "MicroSD Card"
Changed lines of the file:
@@
 	18900 9950 18900 9900
 Connection ~ 18900 9950
-Text Label 19450 9950 0    60   ~ 0
-ALERT
 Wire Wire Line
 	17950 10850 18100 10850
@@
 Text Notes 2750 1150 0    50   ~ 0
 Pin Headers and General Connection Labeling
-$Comp
-L Connector:Micro_SD_Card J1
-U 1 1 5C383B9E
-P 10700 10350
-F 0 "J1" H 10650 9533 50  0000 C CNN
-F 1 "Micro_SD_Card" H 10650 9624 50  0000 C CNN
-F 2 "" H 11850 10650 50  0001 C CNN
-F 3 "http://katalog.we-online.de/em/datasheet/693072010801.pdf" H 10700 10350 50  0001 C CNN
-	1    10700 10350
-	-1   0    0    1
-$EndComp
 Wire Notes Line
 	15400 8250 9150 8250
@@
 	15400 12200 15400 8250
 Wire Wire Line
-	11600 10150 11950 10150
-Wire Wire Line
-	11950 10150 11950 9300
-Wire Wire Line
-	11950 9300 9800 9300
-Wire Wire Line
-	9800 9300 9800 9750
-Wire Wire Line
-	9800 9750 9900 9750
-Wire Wire Line
-	11600 9950 12400 9950
-Wire Wire Line
-	11600 10050 12400 10050
-Text Label 12400 9950 0    50   ~ 0
-DAT1
-Text Label 12400 10050 0    50   ~ 0
-DAT0
-Wire Wire Line
-	11950 9300 12250 9300
-Connection ~ 11950 9300
-Text GLabel 12250 9300 2    60   Input ~ 0
+	13450 9500 13800 9500
+Wire Wire Line
+	13800 9500 13800 8650
+Wire Wire Line
+	13800 8650 13700 8650
+Wire Wire Line
+	11650 8650 11650 9100
+Wire Wire Line
+	11650 9100 11750 9100
+Wire Wire Line
+	13450 9300 14250 9300
+Wire Wire Line
+	13450 9400 14250 9400
+Text Label 14250 9400 0    50   ~ 0
+DAT0_MISO
+Wire Wire Line
+	13800 8650 14100 8650
+Connection ~ 13800 8650
+Text GLabel 14100 8650 2    60   Input ~ 0
 DGND
 Wire Wire Line
-	11600 10250 12700 10250
-Text Label 12700 10250 0    50   ~ 0
+	13450 9600 14550 9600
+Text Label 14550 9600 0    50   ~ 0
 uSD_CLK
 Wire Wire Line
-	13100 10350 13100 9300
-Wire Wire Line
-	11600 10350 13100 10350
-Text GLabel 13100 9300 2    60   Input ~ 0
+	14950 9700 14950 8650
+Wire Wire Line
+	13450 9700 14950 9700
+Text GLabel 14950 8650 2    60   Input ~ 0
 DVDD
 Wire Wire Line
-	11600 10450 12400 10450
-Text Label 12400 10450 0    50   ~ 0
-CMD
-Wire Wire Line
-	11600 10550 12400 10550
-Text Label 12400 10550 0    50   ~ 0
-DAT3
-Wire Wire Line
-	11600 10650 12400 10650
-Text Label 12400 10650 0    50   ~ 0
-DAT2
-Wire Wire Line
-	25050 4800 25550 4800
-Wire Wire Line
-	25550 4800 25550 5400
+	13450 9800 14250 9800
+Text Label 14250 9800 0    50   ~ 0
+CMD_MOSI
+Wire Wire Line
+	13450 9900 14250 9900
+Text Label 14250 9900 0    50   ~ 0
+DAT3_CS
+Wire Wire Line
+	13450 10000 14250 10000
+Text Label 14250 10000 0    50   ~ 0
+DAT2_UNUSED
 Wire Wire Line
 	23400 5700 23400 6250
@@
 Wire Wire Line
 	23600 5700 23600 6250
-Text Label 23400 6250 1    60   ~ 0
-ALERT
 Text Label 23500 6250 1    60   ~ 0
 SCL
 Text Label 23600 6250 1    60   ~ 0
 SDA
+Text Label 24100 6350 1    50   ~ 0
+DAT0_MISO
+Text Label 24200 6350 1    50   ~ 0
+uSD_CLK
+Text Label 24300 6350 1    50   ~ 0
+CMD_MOSI
+Text Label 24400 6350 1    50   ~ 0
+DAT3_CS
+Text Label 14250 9300 0    50   ~ 0
+DAT1_UNUSED
+NoConn ~ 14250 9300
+NoConn ~ 14250 10000
+Wire Wire Line
+	24100 5700 24100 6350
+Wire Wire Line
+	24200 5700 24200 6350
+Wire Wire Line
+	24300 6350 24300 5700
+Wire Wire Line
+	24400 5700 24400 6350
+Text Notes 9150 8250 0    50   ~ 0
+MicroSD Card
+Text Label 23400 6250 1    60   ~ 0
+ALERT
+$Comp
+L Connector:Micro_SD_Card_Det J1
+U 1 1 5C6FB1A7
+P 12550 9600
+F 0 "J1" H 12500 8783 50  0000 C CNN
+F 1 "Micro_SD_Card_Det" H 12500 8874 50  0000 C CNN
+F 2 "" H 14600 10300 50  0001 C CNN
+F 3 "https://www.hirose.com/product/en/download_file/key_name/DM3/category/Catalog/doc_file_id/49662/?file_category_id=4&item_id=195&is_series=1" H 12550 9700 50  0001 C CNN
+	1    12550 9600
+	-1   0    0    1
+$EndComp
+Wire Wire Line
+	13450 9100 13700 9100
+Wire Wire Line
+	13450 9200 13700 9200
+Wire Wire Line
+	13700 8650 13700 9100
+Connection ~ 13700 9100
+Wire Wire Line
+	13700 9100 13700 9200
+Connection ~ 13700 8650
+Wire Wire Line
+	13700 8650 11650 8650
 $EndSCHEMATC

Commit message: Replaced through-hole footprints with pads.
Changed lines of the file:
@@
 Wire Wire Line
 	13700 8650 11650 8650
+Text Label 19450 9950 0    60   ~ 0
+ALERT
 $EndSCHEMATC

Commit message: Updated schematic, and footprints. PCB needs arrangement and routing.
Parts:
- removed R4: 200k, Resistors_SMD:R_0402, symbol Device:R
- added C10, C9: 10uF, Capacitors_SMD:C_0402, symbol Device:C
- added C7, C8: 0.1uF, Capacitors_SMD:C_0402, symbol Device:C
- added IC1: AD5242BRUZ1M, SOP65P640X120-16N, symbol AD5242BRUZ1M:AD5242BRUZ1M
- added L2: 4.7uH, Inductors_SMD:L_0603, symbol conn1:INDUCTOR
- added U7: ADS1220, Package_DFN_QFN:QFN-16-1EP_3x3mm_P0.5mm_EP1.8x1.8mm, symbol bioreactor:ADS1220
- added U8: TPS61222, Package_TO_SOT_SMD:SOT-363_SC-70-6, symbol EEG_ADS1299-cache:TPS61222
Connections:
- net labels added: AD5242_SCL, AD5242_SDA, AD5242_~SHDN, ADC_AIN0, ADC_AIN1, AVDD, DIN, DOUT, RT_1, RT_2, SPI_SCLK, SPI_~CS, TMP_SCL, TMP_SDA, ~DRDY
- net labels removed: GSR_AIN, SCL, SDA
- wire segments 337 -> 413
- no-connect marks 3 -> 14
Other:
- note added: "5.0 V Regulator"
- note added: "ADC"
- note added: "reference"

Commit message: Added switch and arranged and routed PCB.
Parts:
- added S1: SSAJ120100, SSAJ120100, symbol SSAJ120100:SSAJ120100
Connections:
- net labels added: LOAD_OUT, TMP_ALERT
- net labels removed: ALERT
- wire segments 413 -> 438
- no-connect marks 14 -> 15
Other:
- note added: "Digital Potentiometer"
- note added: "Switch"
- note removed: "Vin"
Changed lines of the file:
@@
 Text Notes 13700 1950 0    60   ~ 0
 Vout
-Text Notes 17700 2800 0    60   ~ 0
-Vin
 $Comp
 L conn1:GND-RESCUE-emg_circuit_2_ext_amp #PWR03
@@
 	1    0    0    -1
 $EndComp
-Text Label 6450 1950 2    60   ~ 0
-LOAD_IN
-Text Label 18150 2950 0    60   ~ 0
+Text Label 11100 5550 0    60   ~ 0
 LOAD_IN
 Text GLabel 10800 6050 0    60   Input ~ 0
@@
 	10250 5550 10800 5550
 Connection ~ 10800 5550
-$Comp
-L power:VCC #PWR05
-U 1 1 5B33E296
-P 11100 5550
-F 0 "#PWR05" H 11100 5650 30  0001 C CNN
-F 1 "VCC" H 11100 5650 30  0000 C CNN
-F 2 "" H 11100 5550 60  0000 C CNN
-F 3 "" H 11100 5550 60  0000 C CNN
-	1    11100 5550
-	1    0    0    -1
-$EndComp
 Text Notes 11200 5350 0    60   ~ 0
 TO LOAD
@@
 Text Label 14250 10000 0    50   ~ 0
 DAT2_UNUSED
-Wire Wire Line
-	23400 5700 23400 6250
-Wire Wire Line
-	23500 5700 23500 6250
-Wire Wire Line
-	23600 5700 23600 6250
-Text Label 23500 6250 1    60   ~ 0
+Text Label 24200 6350 1    60   ~ 0
 TMP_SCL
-Text Label 23600 6250 1    60   ~ 0
+Text Label 24300 6350 1    60   ~ 0
 TMP_SDA
-Text Label 24100 6350 1    50   ~ 0
+Text Label 24400 6350 1    50   ~ 0
 DAT0_MISO
-Text Label 24200 6350 1    50   ~ 0
+Text Label 25550 5400 1    50   ~ 0
 uSD_CLK
-Text Label 24300 6350 1    50   ~ 0
+Text Label 25650 5400 1    50   ~ 0
 CMD_MOSI
-Text Label 24400 6350 1    50   ~ 0
+Text Label 25750 5400 1    50   ~ 0
 DAT3_CS
 Text Label 14250 9300 0    50   ~ 0
@@
 Text Notes 9150 8250 0    50   ~ 0
 MicroSD Card
-Text Label 23400 6250 1    60   ~ 0
-ALERT
+Text Label 20450 5050 0    60   ~ 0
+TMP_ALERT
 $Comp
 L Connector:Micro_SD_Card_Det J1
@@
 	13700 8650 11650 8650
 Text Label 19450 9950 0    60   ~ 0
-ALERT
+TMP_ALERT
 $Comp
 L bioreactor:ADS1220 U7
@@
 	14850 4450 14550 4450
 Connection ~ 14850 4450
-Text Label 14400 4450 0    60   ~ 0
-LOAD_IN
 Wire Notes Line
 	13350 4250 18600 4250
@@
 L AD5242BRUZ1M:AD5242BRUZ1M IC1
 U 1 1 5D0D375D
-P 23500 13500
-F 0 "IC1" H 24100 13765 50  0000 C CNN
-F 1 "AD5242BRUZ1M" H 24100 13674 50  0000 C CNN
-F 2 "SOP65P640X120-16N" H 24550 13600 50  0001 L CNN
-F 3 "http://www.mouser.com/datasheet/2/609/AD5241_5242-586728.pdf" H 24550 13500 50  0001 L CNN
-F 4 "AD5242BRUZ1M, Digital Potentiometer 1000k 256-Position 2-channel Serial-2 Wire, Serial-I2C 16-Pin TSSOP" H 24550 13400 50  0001 L CNN "Description"
-F 5 "1.2" H 24550 13300 50  0001 L CNN "Height"
-F 6 "584-AD5242BRUZ1M" H 24550 13200 50  0001 L CNN "Mouser Part Number"
-F 7 "https://www.mouser.com/Search/Refine.aspx?Keyword=584-AD5242BRUZ1M" H 24550 13100 50  0001 L CNN "Mouser Price/Stock"
-F 8 "Analog Devices" H 24550 13000 50  0001 L CNN "Manufacturer_Name"
-F 9 "AD5242BRUZ1M" H 24550 12900 50  0001 L CNN "Manufacturer_Part_Number"
-	1    23500 13500
+P 25650 14100
+F 0 "IC1" H 26250 14365 50  0000 C CNN
+F 1 "AD5242BRUZ1M" H 26250 14274 50  0000 C CNN
+F 2 "SOP65P640X120-16N" H 26700 14200 50  0001 L CNN
+F 3 "http://www.mouser.com/datasheet/2/609/AD5241_5242-586728.pdf" H 26700 14100 50  0001 L CNN
+F 4 "AD5242BRUZ1M, Digital Potentiometer 1000k 256-Position 2-channel Serial-2 Wire, Serial-I2C 16-Pin TSSOP" H 26700 14000 50  0001 L CNN "Description"
+F 5 "1.2" H 26700 13900 50  0001 L CNN "Height"
+F 6 "584-AD5242BRUZ1M" H 26700 13800 50  0001 L CNN "Mouser Part Number"
+F 7 "https://www.mouser.com/Search/Refine.aspx?Keyword=584-AD5242BRUZ1M" H 26700 13700 50  0001 L CNN "Mouser Price/Stock"
+F 8 "Analog Devices" H 26700 13600 50  0001 L CNN "Manufacturer_Name"
+F 9 "AD5242BRUZ1M" H 26700 13500 50  0001 L CNN "Manufacturer_Part_Number"
+	1    25650 14100
 	1    0    0    -1
 $EndComp
@@
 Text Label 24500 10200 0    50   ~ 0
 RT_2
-Text Label 22650 14000 0    50   ~ 0
+Text Label 24800 14600 0    50   ~ 0
 AD5242_~SHDN
 Wire Wire Line
-	22650 14000 23500 14000
-Wire Wire Line
-	23500 13900 22500 13900
-Text GLabel 22500 13450 0    60   Input ~ 0
+	24800 14600 25650 14600
+Wire Wire Line
+	25650 14500 24650 14500
+Text GLabel 24650 14050 0    60   Input ~ 0
 DVDD
 Wire Wire Line
-	23500 13600 23050 13600
-Wire Wire Line
-	23500 13700 22950 13700
-Wire Wire Line
-	22950 13700 22950 13300
-Wire Wire Line
-	23500 13800 22100 13800
-Wire Wire Line
-	22100 13800 22100 14300
-Text GLabel 22100 14300 0    60   Input ~ 0
-DGND
-Wire Wire Line
-	22950 13300 22750 13300
-Wire Wire Line
-	22750 13300 22750 13250
-Text Label 22750 13250 0    50   ~ 0
+	25650 14200 25200 14200
+Wire Wire Line
+	25650 14300 25100 14300
+Wire Wire Line
+	25100 14300 25100 13900
+Wire Wire Line
+	25650 14400 24250 14400
+Wire Wire Line
+	24250 14400 24250 14900
+Text GLabel 24250 14900 0    60   Input ~ 0
+DGND
+Wire Wire Line
+	25100 13900 24900 13900
+Wire Wire Line
+	24900 13900 24900 13850
+Text Label 24900 13850 0    50   ~ 0
 RT_2
 Wire Wire Line
-	22750 13150 22750 13100
-Wire Wire Line
-	23050 13150 23050 13600
-Wire Wire Line
-	22750 13150 23050 13150
-Text Label 22750 13100 0    50   ~ 0
+	24900 13750 24900 13700
+Wire Wire Line
+	25200 13750 25200 14200
+Wire Wire Line
+	24900 13750 25200 13750
+Text Label 24900 13700 0    50   ~ 0
 RT_1
-NoConn ~ 24700 13500
-NoConn ~ 24700 13600
-NoConn ~ 24700 13700
-NoConn ~ 24700 13800
-Wire Wire Line
-	24700 13900 25350 13900
-Wire Wire Line
-	25350 13900 25350 14000
-Text GLabel 25350 14150 2    60   Input ~ 0
-DGND
-Wire Wire Line
-	24700 14000 25350 14000
-Connection ~ 25350 14000
-Wire Wire Line
-	25350 14000 25350 14150
-Wire Wire Line
-	22500 13450 22500 13900
-Wire Wire Line
-	23500 14100 22700 14100
-Wire Wire Line
-	23500 14200 22700 14200
-Text Label 22700 14100 0    50   ~ 0
+NoConn ~ 26850 14100
+NoConn ~ 26850 14200
+NoConn ~ 26850 14300
+NoConn ~ 26850 14400
+Wire Wire Line
+	26850 14500 27500 14500
+Wire Wire Line
+	27500 14500 27500 14600
+Text GLabel 27500 14750 2    60   Input ~ 0
+DGND
+Wire Wire Line
+	26850 14600 27500 14600
+Connection ~ 27500 14600
+Wire Wire Line
+	27500 14600 27500 14750
+Wire Wire Line
+	24650 14050 24650 14500
+Wire Wire Line
+	25650 14700 24850 14700
+Wire Wire Line
+	25650 14800 24850 14800
+Text Label 24850 14700 0    50   ~ 0
 AD5242_SCL
-Text Label 22700 14200 0    50   ~ 0
+Text Label 24850 14800 0    50   ~ 0
 AD5242_SDA
-NoConn ~ 24700 14100
-NoConn ~ 24700 14200
-NoConn ~ 23500 13500
+NoConn ~ 26850 14700
+NoConn ~ 26850 14800
+NoConn ~ 25650 14100
 Text GLabel 17700 3450 2    60   Input ~ 0
 DGND
@@
 Text GLabel 5700 5700 2    60   Input ~ 0
 DGND
+Wire Notes Line
+	28450 12900 28450 15850
+Wire Notes Line
+	28450 15850 23150 15850
+Wire Notes Line
+	23150 15850 23150 12900
+Wire Notes Line
+	23150 12900 28450 12900
+Text Notes 23150 12850 0    50   ~ 0
+Digital Potentiometer
+$Comp
+L SSAJ120100:SSAJ120100 S1
+U 1 1 5C97C155
+P 2900 8350
+F 0 "S1" H 3300 8615 50  0000 C CNN
+F 1 "SSAJ120100" H 3300 8524 50  0000 C CNN
+F 2 "SSAJ120100" H 3550 8450 50  0001 L CNN
+F 3 "https://componentsearchengine.com/Datasheets/1/SSAJ120100.pdf" H 3550 8350 50  0001 L CNN
+F 4 "Slide Switches 1-pole 2-positions Surface Mount Slide Switch SPDT Maintained 10 mA Slide" H 3550 8250 50  0001 L CNN "Description"
+F 5 "" H 3550 8150 50  0001 L CNN "Height"
+F 6 "688-SSAJ120100" H 3550 8050 50  0001 L CNN "Mouser Part Number"
+F 7 "https://www.mouser.com/Search/Refine.aspx?Keyword=688-SSAJ120100" H 3550 7950 50  0001 L CNN "Mouser Price/Stock"
+F 8 "ALPS" H 3550 7850 50  0001 L CNN "Manufacturer_Name"
+F 9 "SSAJ120100" H 3550 7750 50  0001 L CNN "Manufacturer_Part_Number"
+	1    2900 8350
+	1    0    0    -1
+$EndComp
+Text Notes 3100 7950 0    50   ~ 0
+Switch
+Wire Wire Line
+	2050 8350 2900 8350
+Text Label 2050 8350 0    50   ~ 0
+LOAD_IN
+NoConn ~ 2900 8450
+Wire Wire Line
+	2900 8550 2050 8550
+Text Label 2050 8550 0    50   ~ 0
+LOAD_OUT
+Text Label 14400 4450 0    50   ~ 0
+LOAD_OUT
+Text Label 18150 2950 2    50   ~ 0
+LOAD_OUT
+Text Label 6450 1950 2    50   ~ 0
+LOAD_OUT
+Wire Wire Line
+	3700 8350 4050 8350
+Wire Wire Line
+	4050 8350 4050 8450
+Wire Wire Line
+	3700 8450 4050 8450
+Connection ~ 4050 8450
+Wire Wire Line
+	4050 8450 4050 8550
+Text GLabel 4050 8550 2    60   Input ~ 0
+DGND
+Wire Wire Line
+	22650 4600 22100 4600
+Wire Wire Line
+	22100 4600 22100 5050
+Wire Wire Line
+	22100 5050 21050 5050
+Wire Wire Line
+	22650 4700 22150 4700
+Wire Wire Line
+	22150 4700 22150 5150
+Wire Wire Line
+	22150 5150 21050 5150
+Wire Wire Line
+	22650 4800 22200 4800
+Wire Wire Line
+	22200 4800 22200 5250
+Wire Wire Line
+	22200 5250 21050 5250
+Wire Wire Line
+	25050 4800 25550 4800
+Wire Wire Line
+	25550 4800 25550 5400
+Wire Wire Line
+	25050 4700 25650 4700
+Wire Wire Line
+	25650 4700 25650 5400
+Wire Wire Line
+	25750 4600 25750 5400
+Wire Wire Line
+	25050 4600 25750 4600
+Wire Wire Line
+	23400 5700 23400 6350
+Wire Wire Line
+	23500 5700 23500 6350
+Wire Wire Line
+	23600 5700 23600 6350
+Wire Wire Line
+	23700 5700 23700 6350
+Wire Wire Line
+	23800 5700 23800 6350
+Wire Wire Line
+	23900 5700 23900 6350
+Wire Wire Line
+	24000 5700 24000 6350
+Text Label 23400 6350 1    50   ~ 0
+SPI_~CS
+Text Label 23500 6350 1    50   ~ 0
+SPI_SCLK
+Text Label 23600 6350 1    50   ~ 0
+DIN
+Text Label 23700 6350 1    50   ~ 0
+DOUT
+Text Label 23800 6350 1    50   ~ 0
+~DRDY
 $EndSCHEMATC
